File: ISP-HVP-Shield/Rev_2.0/isp_hvp_shield_topor.brd (EAGLE design)
At the start: 50 x 53 mm, 24 parts, among them IC1 ATtiny13/15/25/45/85, IC2 ATtiny24/44/84, IC3 TINY26/261/461/861, IC4 ATtiny2313/4313, IC5 ATMEGA328, IC6 74HCT595D, IC7 MAX662A, Q1 BC858BSMD

Commit message: Sent Gerber files to fab house...
Parts:
- added E$1: (no value), kaibader:KAI-LOGO-M
- added E$2: (no value), kaibader:OSHW-LOGO-S
Other:
- board text added: "Kai C. Bader CC-BY-SA 3.0"
- board text removed: "CC-BY-SA 3.0"
- board text removed: "Kai C. Bader"
Changed lines of the file:
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@@
 <layer number="20" name="Dimension" color="15" fill="1" visible="yes" active="yes"/>
 <layer number="21" name="tPlace" color="7" fill="1" visible="yes" active="yes"/>
-<layer number="22" name="bPlace" color="7" fill="1" visible="no" active="yes"/>
+<layer number="22" name="bPlace" color="7" fill="1" visible="yes" active="yes"/>
 <layer number="23" name="tOrigins" color="15" fill="1" visible="yes" active="yes"/>
 <layer number="24" name="bOrigins" color="15" fill="1" visible="no" active="yes"/>
@@
 <layer number="48" name="Document" color="7" fill="1" visible="no" active="yes"/>
 <layer number="49" name="Reference" color="7" fill="1" visible="no" active="yes"/>
+<layer number="50" name="dxf" color="7" fill="1" visible="no" active="no"/>
 <layer number="51" name="tDocu" color="7" fill="1" visible="yes" active="yes"/>
 <layer number="52" name="bDocu" color="7" fill="1" visible="no" active="yes"/>
+<layer number="53" name="tGND_GNDA" color="7" fill="9" visible="no" active="no"/>
+<layer number="54" name="bGND_GNDA" color="1" fill="9" visible="no" active="no"/>
+<layer number="56" name="wert" color="7" fill="1" visible="no" active="no"/>
+<layer number="90" name="Modules" color="5" fill="1" visible="no" active="no"/>
 <layer number="91" name="Nets" color="2" fill="1" visible="no" active="no"/>
 <layer number="92" name="Busses" color="1" fill="1" visible="no" active="no"/>
@@
 <layer number="97" name="Info" color="7" fill="1" visible="no" active="no"/>
 <layer number="98" name="Guide" color="6" fill="1" visible="no" active="no"/>
+<layer number="151" name="HeatSink" color="7" fill="1" visible="no" active="yes"/>
+<layer number="152" name="_bDocu" color="7" fill="1" visible="yes" active="yes"/>
+<layer number="199" name="Contour" color="7" fill="1" visible="yes" active="yes"/>
+<layer number="200" name="200bmp" color="1" fill="10" visible="no" active="yes"/>
+<layer number="201" name="201bmp" color="2" fill="10" visible="no" active="yes"/>
+<layer number="202" name="202bmp" color="3" fill="10" visible="no" active="yes"/>
+<layer number="203" name="203bmp" color="4" fill="10" visible="no" active="yes"/>
+<layer number="204" name="204bmp" color="5" fill="10" visible="no" active="yes"/>
+<layer number="205" name="205bmp" color="6" fill="10" visible="no" active="yes"/>
+<layer number="206" name="206bmp" color="7" fill="10" visible="no" active="yes"/>
+<layer number="207" name="207bmp" color="8" fill="10" visible="no" active="yes"/>
+<layer number="208" name="208bmp" color="9" fill="10" visible="no" active="yes"/>
+<layer number="209" name="209bmp" color="7" fill="1" visible="no" active="yes"/>
+<layer number="210" name="210bmp" color="7" fill="1" visible="no" active="yes"/>
+<layer number="211" name="211bmp" color="7" fill="1" visible="no" active="yes"/>
+<layer number="212" name="212bmp" color="7" fill="1" visible="no" active="yes"/>
+<layer number="213" name="213bmp" color="7" fill="1" visible="no" active="yes"/>
+<layer number="214" name="214bmp" color="7" fill="1" visible="no" active="yes"/>
+<layer number="215" name="215bmp" color="7" fill="1" visible="no" active="yes"/>
+<layer number="216" name="216bmp" color="7" fill="1" visible="no" active="yes"/>
+<layer number="217" name="217bmp" color="18" fill="1" visible="no" active="no"/>
+<layer number="218" name="218bmp" color="19" fill="1" visible="no" active="no"/>
+<layer number="219" name="219bmp" color="20" fill="1" visible="no" active="no"/>
+<layer number="220" name="220bmp" color="21" fill="1" visible="no" active="no"/>
+<layer number="221" name="221bmp" color="22" fill="1" visible="no" active="no"/>
+<layer number="222" name="222bmp" color="23" fill="1" visible="no" active="no"/>
+<layer number="223" name="223bmp" color="24" fill="1" visible="no" active="no"/>
+<layer number="224" name="224bmp" color="25" fill="1" visible="no" active="no"/>
+<layer number="248" name="Housing" color="7" fill="1" visible="yes" active="yes"/>
+<layer number="249" name="Edge" color="7" fill="1" visible="yes" active="yes"/>
 <layer number="250" name="Descript" color="3" fill="1" visible="no" active="no"/>
 <layer number="251" name="SMDround" color="12" fill="11" visible="no" active="no"/>
@@
 <layer number="145" name="Edge" color="15" fill="1" visible="yes" active="yes"/>
 <layer number="146" name="cooling" color="15" fill="1" visible="yes" active="yes"/>
+<layer number="254" name="cooling" color="7" fill="1" visible="no" active="yes"/>
 </layers>
 <board>
@@
 <wire x1="50" y1="51" x2="48" y2="53" width="0.001" layer="20" curve="90"/>
 <wire x1="2" y1="53" x2="0" y2="51" width="0.001" layer="20" curve="90"/>
-<text x="6.591" y="14.081" size="1.77798125" layer="21" rot="SR90">ISP/HVP Shield</text>
-<text x="6.463" y="37.719" size="1.016" layer="21" rot="SR90">(Rev 2.0)</text>
-<text x="30.622" y="36.941" size="1.016" layer="21" rot="SR90" align="center-left">CC-BY-SA 3.0</text>
-<text x="30.734" y="23.749" size="1.016" layer="21" rot="SR90" align="center-left">Kai C. Bader</text>
-<text x="20.193" y="5.08" size="1.016" layer="21" rot="SR0" align="center">1+2 = ISP
+<text x="6.591" y="14.589" size="1.77798125" layer="21" rot="SR90">ISP/HVP Shield</text>
+<text x="5.701" y="35.941" size="1.016" layer="21" ratio="10" rot="SR90">(Rev 2.0)</text>
+<text x="30.734" y="23.241" size="1.016" layer="21" ratio="10" rot="SR90" align="center-left">Kai C. Bader    CC-BY-SA 3.0</text>
+<text x="16.129" y="5.08" size="1.016" layer="21" ratio="10" rot="SR0" align="center-left">1+2 = ISP
 2+3 = HVP</text>
+<text x="30.734" y="47.625" size="1.016" layer="22" ratio="10" rot="SMR270" align="center-left">Kai C. Bader    CC-BY-SA 3.0</text>
+<text x="5.955" y="21.971" size="1.016" layer="22" ratio="10" rot="SMR270">(Rev 2.0)</text>
+<text x="6.845" y="43.323" size="1.77798125" layer="22" rot="SMR270">ISP/HVP Shield</text>
 </plain>
 <attributes>
@@
 </class>
 </classes>
-<designrules name="SeeedStudio_2layer_DRU_no_angle_20140221">
+<designrules name="ITEADstudio_DRC">
 <description language="de">&lt;b&gt;EAGLE Design Rules&lt;/b&gt;
 &lt;p&gt;
@@
 </description>
 <param name="layerSetup" value="(1*16)"/>
-<param name="mtCopper" value="0.035mm 0.0175mm 0.035mm 0.035mm 0.035mm 0.035mm 0.035mm 0.035mm 0.035mm 0.035mm 0.035mm 0.035mm 0.035mm 0.035mm 0.0175mm 0.035mm"/>
-<param name="mtIsolate" value="1.5mm 1.1mm 0.2mm 0.15mm 0.2mm 0.15mm 0.2mm 0.15mm 0.2mm 0.15mm 0.2mm 0.15mm 0.2mm 0.15mm 0.2mm"/>
+<param name="mtCopper" value="0.035mm 0.035mm 0.035mm 0.035mm 0.035mm 0.035mm 0.035mm 0.035mm 0.035mm 0.035mm 0.035mm 0.035mm 0.035mm 0.035mm 0.035mm 0.035mm"/>
+<param name="mtIsolate" value="1.5mm 0.15mm 0.2mm 0.15mm 0.2mm 0.15mm 0.2mm 0.15mm 0.2mm 0.15mm 0.2mm 0.15mm 0.2mm 0.15mm 0.2mm"/>
 <param name="mdWireWire" value="6mil"/>
 <param name="mdWirePad" value="6mil"/>
@@
 <attribute name="VALUE" x="6.985" y="3.175" size="1.27001875" layer="27"/>
 </element>
+<element name="E$1" library="kaibader" package="KAI-LOGO-M" value="" x="48.514" y="8.128" rot="R90"/>
+<element name="E$2" library="kaibader" package="OSHW-LOGO-S" value="" x="46.99" y="6.096" rot="R90"/>
 </elements>
 <signals>
